Commit message: Add exploration/sensor_fusion/find_object

File: dhex_description/urdf/attachments.xacro (robot description, xacro)
@@ -1,30 +1,26 @@
 <?xml version="1.0" encoding="utf-8"?>
-<robot xmlns:xacro="http://www.ros.org/wiki/xacro" name="borg_workbench">
-  <link name ="world">
-  </link>
-    <xacro:include filename="$(find borg_arm_description)/urdf/borg_arm.urdf.xacro"/>
-    <xacro:include filename="$(find borg_arm_description)/urdf/borg_camera.urdf.xacro"/>
-    <xacro:include filename="$(find borg_arm_gazebo)/urdf/workbench.urdf.xacro"/>
-    <xacro:include filename="$(find borg_arm_gazebo)/urdf/arm_workspace.urdf.xacro"/>
-    <!-- <xacro:include filename="$(find borg_arm_gazebo)/urdf/box.urdf.xacro"/> -->
-    <joint name="workbench_TO_world" type="fixed">
-      <parent link="world"/>
-      <child link="workbench"/>
-      <origin rpy="0 0 0" xyz="0.0 0.0 -0.10"/>
+<robot xmlns:xacro="http://www.ros.org/wiki/xacro" name="attachments">
+<xacro:arg name="rp_lidar_a1" default="true"/>
+<xacro:property name="rp_lidar_a1" value="$(arg rp_lidar_a1)" />
+	<!-- RP Lidar A1 -->
+	<xacro:if value="${rp_lidar_a1}">
+		<xacro:include filename="$(find dhex_description)/urdf/sensors/rp_lidar_a1.xacro"/>
+    <joint name="{link_00_name}_TO_rp_lidar_A1" type="fixed">
+    <origin xyz="0.02 0 0.055" rpy="0.0 -0.025 0.0"/>
+    <parent link="${link_00_name}"/>
+    <child link="rp_lidar_A1"/>
     </joint>
-    <joint name ="borg_arm_TO_workbench" type="fixed">
-        <origin rpy="0 0 1.5707" xyz="0 -0.58 1.39"/>
-        <parent link="workbench"/>
-        <child link = "${base_link}"/>
-    </joint>
-    <!-- <joint name ="box_TO_workbench" type="fixed">
-        <origin rpy="0 0 0" xyz="0 0.5 0.895"/>
-        <parent link="workbench"/>
-        <child link = "box_base_link"/>
-    </joint> -->
-    <joint name ="arm_workspace_TO_workbench" type="fixed">
-        <origin rpy="0 0 0" xyz="0 -0.58 1.39"/>
-        <parent link="workbench"/>
-        <child link = "arm_workspace"/>
-    </joint>
+	</xacro:if>
+<xacro:include filename="$(find dhex_description)/urdf/sensors/generic_camera.xacro" />
+<generic_camera name="dhex_camera"
+        origin_rpy_i="0 0 0" origin_xyz_i="-0.00000185 -0.00008975 0.00737255"
+        mass="0.00615422"
+        ixx="7.472e-7" ixy="0" ixz="0"
+        iyy="7.6e-7" iyz="0"
+        izz="7.4e-7"
+        meshfile="package://dhex_description/meshes/camera_new.dae"
+        meshscale="1 1 1"
+        parent="${link_00_name}"
+        origin_rpy_j="0 0 0" origin_xyz_j="0.1 0 0.021"
+        />
 </robot>

File: dhex_description/urdf/dhex.urdf.xacro (robot description, xacro)
@@ -1,4 +1,6 @@
 <?xml version="1.0" ?>
 <robot xmlns:xacro="http://www.ros.org/wiki/xacro" name="dhex">
+<!-- <xacro:arg name="rp_lidar_a1" default="true"/>
+<xacro:property name="rp_lidar_a1" value="$(arg rp_lidar_a1)" /> -->
 <!-- BGN - Include -->
 <xacro:include filename="$(find dhex_description)/urdf/dhex_parameters.xacro" />
@@ -94,6 +96,9 @@
         meshfile="package://dhex_description/meshes/caster_wheel.stl"
         meshscale="1 1 1" />
+<!-- ATTACHMENTS	 -->
+<xacro:include filename="$(find dhex_description)/urdf/attachments.xacro" />
 	<gazebo>
 		<!-- <plugin name="gazebo_ros_control" filename="libgazebo_ros_control.so">
+			<robotNamespace>/</robotNamespace>
 		</plugin> -->
 		<plugin name="gazebo_ros_control" filename="libgazebo_ros_diff_drive.so">
@@ -107,23 +112,31 @@
 			<wheelSeparation>0.1275</wheelSeparation>
 			<wheelDiameter>0.06599749</wheelDiameter>
-			<torque>20</torque>
-			<commandTopic>/dhex/cmd_vel</commandTopic>
-			<odometryTopic>/dhex/odom</odometryTopic>
+			<torque>10</torque>
+			<commandTopic>cmd_vel</commandTopic>
+			<odometryTopic>dhex_velocity_controller/odom</odometryTopic>
 			<odometryFrame>odom</odometryFrame>
-			<publishWheelTF>true</publishWheelTF>
-			<publishOdomTF>true</publishOdomTF>
+			<publishWheelTF>false</publishWheelTF>
+			<publishOdomTF>false</publishOdomTF>
 			<publishWheelJointState>true</publishWheelJointState>
-			<robotBaseFrame>${base_link}</robotBaseFrame>
+			<robotBaseFrame>${link_00_name}</robotBaseFrame>
 		</plugin>
-                  <plugin name="p3d_base_controller" filename="libgazebo_ros_p3d.so">
+                <plugin name="imu_plugin" filename="libgazebo_ros_imu.so">
                         <alwaysOn>true</alwaysOn>
-                        <updateRate>50.0</updateRate>
-                        <bodyName>base_link</bodyName>
-                        <topicName>ground_truth/state</topicName>
-                        <gaussianNoise>0.01</gaussianNoise>
-                        <frameName>map</frameName>
-                        <xyzOffset>0 0 0</xyzOffset>
-                        <rpyOffset>0 0 0</rpyOffset>
+                        <bodyName>${link_00_name}</bodyName>
+                        <topicName>imu</topicName>
+                        <serviceName>imu_service</serviceName>
+                        <gaussianNoise>0.0</gaussianNoise>
+                        <updateRate>240.0</updateRate>
                 </plugin>
+		<plugin name="p3d_base_controller" filename="libgazebo_ros_p3d.so">
+					<alwaysOn>true</alwaysOn>
+					<updateRate>50.0</updateRate>
+					<bodyName>${link_00_name}</bodyName>
+					<topicName>ground_truth/state</topicName>
+					<gaussianNoise>0.01</gaussianNoise>
+					<frameName>map</frameName>
+					<xyzOffset>0 0 0</xyzOffset>
+					<rpyOffset>0 0 0</rpyOffset>
+		</plugin>
 	</gazebo>
 </robot>

File: dhex_description/urdf/dhex_parameters.xacro (robot description, xacro)
@@ -2,5 +2,5 @@
 <robot xmlns:xacro="http://www.ros.org/wiki/xacro">
   <xacro:property name="base_link" value="base_link" />
-  <xacro:property name="link_00_name" value="dhex_base_link" />
+  <xacro:property name="link_00_name" value="dhex_chassis" />
   <xacro:property name="link_01_name" value="right_wheel" />
   <xacro:property name="link_02_name" value="left_wheel" />

File: dhex_description/urdf/links_joints.xacro (robot description, xacro)
@@ -14,8 +14,8 @@
       <type>transmission_interface/SimpleTransmission</type>
       <joint name="${name}">
-        <hardwareInterface>hardware_interface/PositionJointInterface</hardwareInterface>
+        <hardwareInterface>hardware_interface/EffortJointInterface</hardwareInterface>
       </joint>
       <actuator name="motor_${name}">
-        <hardwareInterface>hardware_interface/PositionJointInterface</hardwareInterface>
+        <hardwareInterface>hardware_interface/EffortJointInterface</hardwareInterface>
         <mechanicalReduction>1</mechanicalReduction>
       </actuator>

File: dhex_description/urdf/sensors/dhex_camera.urdf.xacro (robot description, xacro)
@@ -1,8 +1,9 @@
 <?xml version="1.0" ?>
-<robot xmlns:xacro="http://www.ros.org/wiki/xacro" name="hex_camera">
+<robot xmlns:xacro="http://www.ros.org/wiki/xacro" name="dhex_camera">
   <!-- BGN - Include -->
-  <xacro:include filename="$(find dhex_description)/urdf/generic_camera.xacro" />
+  <xacro:include filename="$(find dhex_description)/urdf/sensors/generic_camera.xacro" />
   <!-- END - Include -->
-<generic_camera name="hex_camera"
+<link name="base_link"/>
+<generic_camera name="dhex_camera"
         origin_rpy_i="0 0 0" origin_xyz_i="-0.08296871 0.00060854 0.00007174"
         mass="0.07334031"
@@ -12,8 +13,6 @@
         meshfile="package://dhex_description/meshes/camera_new.stl"
         meshscale="1 1 1"
-        parent="CAMERA_HOLDER"
+        parent="base_link"
         origin_rpy_j="0 0 1.5707" origin_xyz_j="0 0.08028694 0.0065"
-        px_width="2592"
-        px_heigth="2048"
         />
 </robot>

File: dhex_description/urdf/sensors/generic_camera.xacro (robot description, xacro)
@@ -8,9 +8,9 @@
                        topic:=/camera
                        hz:=30
-                       fov:=${M_PI/2.0}
-                       px_width:=1280
-                       px_heigth:=720
+                       fov:=${60.0*M_PI/180.0}
+                       px_width:=640
+                       px_heigth:=480
                        px_format:=R8G8B8
-                       clip_near:=0.02
+                       clip_near:=0.05
                        clip_far:=300
                        noise:=0.008
@@ -52,5 +52,4 @@
           <mesh filename="${meshfile}" scale="${meshscale}"/>
         </geometry>
-        <material name="light_black"/>
       </visual>
     </link>
@@ -68,7 +67,4 @@
       <child link="${name}_optical_frame"/>
     </joint>
-    <gazebo reference="${name}">
-      <material>Gazebo/Red</material>
-    </gazebo>
     <gazebo reference="${name}">
       <sensor type="camera" name="${name}_sensor">
