Commit message: Add ros_control to wheel joints

File: dhex_description/urdf/dhex.urdf.xacro (robot description, xacro)
@@ -1,101 +1,101 @@
 <?xml version="1.0" ?>
 <robot xmlns:xacro="http://www.ros.org/wiki/xacro" name="dhex">
-<!-- BGN - Include -->
-<xacro:include filename="$(find dhex_description)/urdf/dhex_parameters.xacro" />
-<xacro:include filename="$(find dhex_description)/urdf/links_joints.xacro" />
-<!-- END - Include -->
-<!-- BGN - Robot description -->
-<!-- BASE  -->
-<link name="${base_link}"/>
- <!-- JOINT - BASE_LINK TO HEX_BASE_LINK -->
-<m_joint name="${base_link}_TO_${link_00_name}" type="fixed"
-        axis_xyz="0 0 1"
-        origin_rpy="0 0 0" origin_xyz="0 0 0"
-        parent="${base_link}" child="${link_00_name}"
-        limit_e="1000" limit_l="-3.14" limit_u="3.14" limit_v="0.5" />
-<!-- HEX_BASE_LINK  -->
-<m_link_mesh name="${link_00_name}"
-        origin_rpy_i="0 0 0" origin_xyz_i="0.00643363 -0.00003738 0.00608448"
-        origin_rpy_c="0 0 0" origin_xyz_c="0 0 0"
-        origin_rpy_v = "0 0 0" origin_xyz_v ="0 0 0"
-        mass="0.27625906"
-        ixx="0.0003358" ixy="2.321e-6" ixz="-3.063e-5"
-        iyy="0.00073197" iyz="0.00000108"
-        izz="0.00089429"
-        meshfile="package://dhex_description/meshes/dhex_base_link.dae"
-        meshscale="1 1 1" />
-<!-- JOINT - HEX_BASE_LINK TO RIGHT_WHEEL -->
-<m_joint name="${link_00_name}_TO_${link_01_name}" type="continuous"
-            axis_xyz="0 0 -1"
-            origin_rpy="1.5707 0 0" origin_xyz="0.04739898 -0.06196184 -0.01215966"
-            parent="${link_00_name}" child="${link_01_name}"
-            limit_e="1000" limit_l="-3.14" limit_u="3.14" limit_v="0.5" />
-<!-- RIGHT_WHEEL  -->
-<m_link_mesh name="${link_01_name}"
-        origin_rpy_i="0 0 0" origin_xyz_i="0 0 0"
-        origin_rpy_c="0 0 0" origin_xyz_c="0 0 0"
-        origin_rpy_v = "0 0 0" origin_xyz_v ="0 0 0"
-        mass="0.02990224"
-        ixx="0.00001354" ixy="0" ixz="0"
-        iyy="0.00001354" iyz="0"
-        izz="0.00002032"
-        meshfile="package://dhex_description/meshes/wheel.dae"
-        meshscale="1 1 1" />
-		<!-- origin_rpy_i="0 0 0" origin_xyz_i="0.04318327 -0.06196513 -0.0084928" -->
-<!-- JOINT - HEX_BASE_LINK TO LEFT_WHEEL -->
-<m_joint name="${link_00_name}_TO_${link_02_name}" type="continuous"
-            axis_xyz="0 0 1"
-            origin_rpy="-1.5707 0 0" origin_xyz="0.04739898 0.06196184 -0.01215966"
-            parent="${link_00_name}" child="${link_02_name}"
-            limit_e="1000" limit_l="-3.14" limit_u="3.14" limit_v="0.5" />
-<!--LEFT_WHEEL-->
-<m_link_mesh name="${link_02_name}"
-        origin_rpy_i="0 0 0" origin_xyz_i="0.0 0.0 0.0"
-        origin_rpy_c="0 0 0" origin_xyz_c="0 0 0"
-        origin_rpy_v = "0 0 0" origin_xyz_v ="0 0 0"
-        mass="0.02990224"
-        ixx="0.00001354" ixy="0" ixz="0"
-        iyy="0.00001354" iyz="0"
-        izz="0.00002032"
-        meshfile="package://dhex_description/meshes/wheel.dae"
-        meshscale="1 1 1" />
-<!-- JOINT - HEX_BASE_LINK TO CASTER_WHEEL_SUPPORT -->
-<m_joint name="${link_00_name}_TO_${link_03_name}" type="continuous"
-            axis_xyz="0 0 1"
-            origin_rpy="0 0 0" origin_xyz="-0.06827047 0.00004137 -0.03548239"
-            parent="${link_00_name}" child="${link_03_name}"
-            limit_e="1000" limit_l="-3.14" limit_u="3.14" limit_v="0.5" />
-<!--CASTER_WHEEL_SUPPORT-->
-<m_link_mesh name="${link_03_name}"
-        origin_rpy_i="0 0 0" origin_xyz_i="-0.00046976 -0.00666343 0.01149424"
-        origin_rpy_c="0 0 0" origin_xyz_c="0 0 0"
-        origin_rpy_v = "0 0 0" origin_xyz_v ="0 0 0"
-        mass="0.01744074 "
-        ixx="0.00000232" ixy="-7.239e-8" ixz="-9.416e-8"
-        iyy="0.00000226" iyz="-7.1e-7"
-        izz="0.0000025"
-        meshfile="package://dhex_description/meshes/caster_wheel_support.stl"
-        meshscale="1 1 1" />
-<!-- JOINT - HEX_BASE_LINK TO CASTER_WHEEL -->
-<m_joint name="${link_03_name}_TO_${link_04_name}" type="continuous"
-            axis_xyz="0 0 1"
-            origin_rpy="0 1.5707 0" origin_xyz="0 -0.0155 0"
-            parent="${link_03_name}" child="${link_04_name}"
-            limit_e="1000" limit_l="-3.14" limit_u="3.14" limit_v="0.5" />
-<!--CASTER_WHEEL-->
-<m_link_mesh name="${link_04_name}"
-        origin_rpy_i="0 0 0" origin_xyz_i="0.0 0.0 0.0"
-        origin_rpy_c="0 0 0" origin_xyz_c="0 0 0"
-        origin_rpy_v = "0 0 0" origin_xyz_v ="0 0 0"
-        mass="0.00473765"
-        ixx="2.659e-7" ixy="0" ixz="0"
-        iyy="2.659e-7" iyz="0"
-        izz="4.200e-7"
-        meshfile="package://dhex_description/meshes/caster_wheel.stl"
-        meshscale="1 1 1" />
-	<gazebo>
+  <!-- BGN - Include -->
+  <xacro:include filename="$(find dhex_description)/urdf/dhex_parameters.xacro" />
+  <xacro:include filename="$(find dhex_description)/urdf/links_joints.xacro" />
+  <!-- END - Include -->
+  <!-- BGN - Robot description -->
+  <!-- BASE  -->
+  <link name="${base_link}"/>
+  <!-- JOINT - BASE_LINK TO HEX_BASE_LINK -->
+  <m_joint name="${base_link}_TO_${link_00_name}" type="fixed"
+    axis_xyz="0 0 1"
+    origin_rpy="0 0 0" origin_xyz="0 0 0"
+    parent="${base_link}" child="${link_00_name}"
+    limit_e="1000" limit_l="-3.14" limit_u="3.14" limit_v="0.5" />
+  <!-- HEX_BASE_LINK  -->
+  <m_link_mesh name="${link_00_name}"
+    origin_rpy_i="0 0 0" origin_xyz_i="0.00643363 -0.00003738 0.00608448"
+    origin_rpy_c="0 0 0" origin_xyz_c="0 0 0"
+    origin_rpy_v = "0 0 0" origin_xyz_v ="0 0 0"
+    mass="0.27625906"
+    ixx="0.0003358" ixy="2.321e-6" ixz="-3.063e-5"
+    iyy="0.00073197" iyz="0.00000108"
+    izz="0.00089429"
+    meshfile="package://dhex_description/meshes/dhex_base_link.dae"
+    meshscale="1 1 1" />
+  <!-- JOINT - HEX_BASE_LINK TO RIGHT_WHEEL -->
+  <m_joint name="${link_00_name}_TO_${link_01_name}" type="continuous"
+    axis_xyz="0 0 -1"
+    origin_rpy="1.5707 0 0" origin_xyz="0.04739898 -0.06196184 -0.01215966"
+    parent="${link_00_name}" child="${link_01_name}"
+    limit_e="1000" limit_l="-3.14" limit_u="3.14" limit_v="0.5" />
+  <!-- RIGHT_WHEEL  -->
+  <m_link_mesh name="${link_01_name}"
+    origin_rpy_i="0 0 0" origin_xyz_i="0 0 0"
+    origin_rpy_c="0 0 0" origin_xyz_c="0 0 0"
+    origin_rpy_v = "0 0 0" origin_xyz_v ="0 0 0"
+    mass="0.02990224"
+    ixx="0.00001354" ixy="0" ixz="0"
+    iyy="0.00001354" iyz="0"
+    izz="0.00002032"
+    meshfile="package://dhex_description/meshes/wheel.dae"
+    meshscale="1 1 1" />
+    <!-- origin_rpy_i="0 0 0" origin_xyz_i="0.04318327 -0.06196513 -0.0084928" -->
+  <!-- JOINT - HEX_BASE_LINK TO LEFT_WHEEL -->
+  <m_joint name="${link_00_name}_TO_${link_02_name}" type="continuous"
+    axis_xyz="0 0 1"
+    origin_rpy="-1.5707 0 0" origin_xyz="0.04739898 0.06196184 -0.01215966"
+    parent="${link_00_name}" child="${link_02_name}"
+    limit_e="1000" limit_l="-3.14" limit_u="3.14" limit_v="0.5" />
+  <!--LEFT_WHEEL-->
+  <m_link_mesh name="${link_02_name}"
+    origin_rpy_i="0 0 0" origin_xyz_i="0.0 0.0 0.0"
+    origin_rpy_c="0 0 0" origin_xyz_c="0 0 0"
+    origin_rpy_v = "0 0 0" origin_xyz_v ="0 0 0"
+    mass="0.02990224"
+    ixx="0.00001354" ixy="0" ixz="0"
+    iyy="0.00001354" iyz="0"
+    izz="0.00002032"
+    meshfile="package://dhex_description/meshes/wheel.dae"
+    meshscale="1 1 1" />
+  <!-- JOINT - HEX_BASE_LINK TO CASTER_WHEEL_SUPPORT -->
+  <m_joint name="${link_00_name}_TO_${link_03_name}" type="continuous"
+    axis_xyz="0 0 1"
+    origin_rpy="0 0 0" origin_xyz="-0.06827047 0.00004137 -0.03548239"
+    parent="${link_00_name}" child="${link_03_name}"
+    limit_e="1000" limit_l="-3.14" limit_u="3.14" limit_v="0.5" />
+  <!--CASTER_WHEEL_SUPPORT-->
+  <m_link_mesh name="${link_03_name}"
+    origin_rpy_i="0 0 0" origin_xyz_i="-0.00046976 -0.00666343 0.01149424"
+    origin_rpy_c="0 0 0" origin_xyz_c="0 0 0"
+    origin_rpy_v = "0 0 0" origin_xyz_v ="0 0 0"
+    mass="0.01744074 "
+    ixx="0.00000232" ixy="-7.239e-8" ixz="-9.416e-8"
+    iyy="0.00000226" iyz="-7.1e-7"
+    izz="0.0000025"
+    meshfile="package://dhex_description/meshes/caster_wheel_support.stl"
+    meshscale="1 1 1" />
+  <!-- JOINT - HEX_BASE_LINK TO CASTER_WHEEL -->
+  <m_joint name="${link_03_name}_TO_${link_04_name}" type="continuous"
+    axis_xyz="0 0 1"
+    origin_rpy="0 1.5707 0" origin_xyz="0 -0.0155 0"
+    parent="${link_03_name}" child="${link_04_name}"
+    limit_e="1000" limit_l="-3.14" limit_u="3.14" limit_v="0.5" />
+  <!--CASTER_WHEEL-->
+  <m_link_mesh name="${link_04_name}"
+    origin_rpy_i="0 0 0" origin_xyz_i="0.0 0.0 0.0"
+    origin_rpy_c="0 0 0" origin_xyz_c="0 0 0"
+    origin_rpy_v = "0 0 0" origin_xyz_v ="0 0 0"
+    mass="0.00473765"
+    ixx="2.659e-7" ixy="0" ixz="0"
+    iyy="2.659e-7" iyz="0"
+    izz="4.200e-7"
+    meshfile="package://dhex_description/meshes/caster_wheel.stl"
+    meshscale="1 1 1" />
+  <gazebo>
 		<!-- <plugin name="gazebo_ros_control" filename="libgazebo_ros_control.so">
 		</plugin> -->
-		<plugin name="gazebo_ros_control" filename="libgazebo_ros_diff_drive.so">
+		<!-- <plugin name="gazebo_ros_control" filename="libgazebo_ros_diff_drive.so">
 			<robotNamespace>/</robotNamespace>
 			<legacyModeNS>true</legacyModeNS>
@@ -116,14 +116,14 @@
 			<robotBaseFrame>${base_link}</robotBaseFrame>
 		</plugin>
-                  <plugin name="p3d_base_controller" filename="libgazebo_ros_p3d.so">
-                        <alwaysOn>true</alwaysOn>
-                        <updateRate>50.0</updateRate>
-                        <bodyName>base_link</bodyName>
-                        <topicName>ground_truth/state</topicName>
-                        <gaussianNoise>0.01</gaussianNoise>
-                        <frameName>map</frameName>
-                        <xyzOffset>0 0 0</xyzOffset>
-                        <rpyOffset>0 0 0</rpyOffset>
-                </plugin>
+    <plugin name="p3d_base_controller" filename="libgazebo_ros_p3d.so">
+      <alwaysOn>true</alwaysOn>
+      <updateRate>50.0</updateRate>
+      <bodyName>base_link</bodyName>
+      <topicName>ground_truth/state</topicName>
+      <gaussianNoise>0.01</gaussianNoise>
+      <frameName>map</frameName>
+      <xyzOffset>0 0 0</xyzOffset>
+      <rpyOffset>0 0 0</rpyOffset>
+    </plugin> -->
 	</gazebo>
 </robot>

File: dhex_description/urdf/links_joints.xacro (robot description, xacro)
@@ -1,5 +1,5 @@
 <?xml version="1.0" ?>
 <robot xmlns:xacro="http://www.ros.org/wiki/xacro">
-  <xacro:macro name="m_joint" params="name type axis_xyz origin_rpy origin_xyz parent child limit_e limit_l limit_u limit_v">
+  <xacro:macro name="m_joint" params="name type motor_flag:=false axis_xyz origin_rpy origin_xyz parent child limit_e limit_l limit_u limit_v">
     <joint name="${name}" type="${type}">
       <axis xyz="${axis_xyz}" />
@@ -9,16 +9,29 @@
       <child link="${child}" />
     </joint>
-  <xacro:property name="joint_type" value="revolute"/>
-  <xacro:if value="${joint_type == type}">
-    <transmission name="trans_${name}">
-      <type>transmission_interface/SimpleTransmission</type>
-      <joint name="${name}">
-        <hardwareInterface>hardware_interface/PositionJointInterface</hardwareInterface>
-      </joint>
-      <actuator name="motor_${name}">
-        <hardwareInterface>hardware_interface/PositionJointInterface</hardwareInterface>
-        <mechanicalReduction>1</mechanicalReduction>
-      </actuator>
-    </transmission>
+  <xacro:if value="${motor_flag == 'true'}">
+    <xacro:if value="${joint_type == 'revolute'}">
+      <transmission name="trans_${name}">
+        <type>transmission_interface/SimpleTransmission</type>
+        <joint name="${name}">
+          <hardwareInterface>hardware_interface/PositionJointInterface</hardwareInterface>
+        </joint>
+        <actuator name="motor_${name}">
+          <hardwareInterface>hardware_interface/PositionJointInterface</hardwareInterface>
+          <mechanicalReduction>1</mechanicalReduction>
+        </actuator>
+      </transmission>
+    </xacro:if>
+    <xacro:if value="${joint_type == 'continuous'}">
+      <transmission name="trans_${name}">
+        <type>transmission_interface/SimpleTransmission</type>
+        <joint name="${name}">
+          <hardwareInterface>hardware_interface/VelocityJointInterface</hardwareInterface>
+        </joint>
+        <actuator name="motor_${name}">
+          <hardwareInterface>hardware_interface/VelocityJointInterface</hardwareInterface>
+          <mechanicalReduction>1</mechanicalReduction>
+        </actuator>
+      </transmission>
+    </xacro:if>
   </xacro:if>
   </xacro:macro>

Commit message: Update xacro to enable ros noetic usage

File: dhex_description/urdf/dhex.urdf.xacro (robot description, xacro)
@@ -1,129 +1,96 @@
 <?xml version="1.0" ?>
 <robot xmlns:xacro="http://www.ros.org/wiki/xacro" name="dhex">
-  <!-- BGN - Include -->
-  <xacro:include filename="$(find dhex_description)/urdf/dhex_parameters.xacro" />
-  <xacro:include filename="$(find dhex_description)/urdf/links_joints.xacro" />
-  <!-- END - Include -->
-  <!-- BGN - Robot description -->
-  <!-- BASE  -->
-  <link name="${base_link}"/>
-  <!-- JOINT - BASE_LINK TO HEX_BASE_LINK -->
-  <m_joint name="${base_link}_TO_${link_00_name}" type="fixed"
-    axis_xyz="0 0 1"
-    origin_rpy="0 0 0" origin_xyz="0 0 0"
-    parent="${base_link}" child="${link_00_name}"
-    limit_e="1000" limit_l="-3.14" limit_u="3.14" limit_v="0.5" />
-  <!-- HEX_BASE_LINK  -->
-  <m_link_mesh name="${link_00_name}"
-    origin_rpy_i="0 0 0" origin_xyz_i="0.00643363 -0.00003738 0.00608448"
-    origin_rpy_c="0 0 0" origin_xyz_c="0 0 0"
-    origin_rpy_v = "0 0 0" origin_xyz_v ="0 0 0"
-    mass="0.27625906"
-    ixx="0.0003358" ixy="2.321e-6" ixz="-3.063e-5"
-    iyy="0.00073197" iyz="0.00000108"
-    izz="0.00089429"
-    meshfile="package://dhex_description/meshes/dhex_base_link.dae"
-    meshscale="1 1 1" />
-  <!-- JOINT - HEX_BASE_LINK TO RIGHT_WHEEL -->
-  <m_joint name="${link_00_name}_TO_${link_01_name}" type="continuous"
-    axis_xyz="0 0 -1"
-    origin_rpy="1.5707 0 0" origin_xyz="0.04739898 -0.06196184 -0.01215966"
-    parent="${link_00_name}" child="${link_01_name}"
-    limit_e="1000" limit_l="-3.14" limit_u="3.14" limit_v="0.5" />
-  <!-- RIGHT_WHEEL  -->
-  <m_link_mesh name="${link_01_name}"
-    origin_rpy_i="0 0 0" origin_xyz_i="0 0 0"
-    origin_rpy_c="0 0 0" origin_xyz_c="0 0 0"
-    origin_rpy_v = "0 0 0" origin_xyz_v ="0 0 0"
-    mass="0.02990224"
-    ixx="0.00001354" ixy="0" ixz="0"
-    iyy="0.00001354" iyz="0"
-    izz="0.00002032"
-    meshfile="package://dhex_description/meshes/wheel.dae"
-    meshscale="1 1 1" />
-    <!-- origin_rpy_i="0 0 0" origin_xyz_i="0.04318327 -0.06196513 -0.0084928" -->
-  <!-- JOINT - HEX_BASE_LINK TO LEFT_WHEEL -->
-  <m_joint name="${link_00_name}_TO_${link_02_name}" type="continuous"
-    axis_xyz="0 0 1"
-    origin_rpy="-1.5707 0 0" origin_xyz="0.04739898 0.06196184 -0.01215966"
-    parent="${link_00_name}" child="${link_02_name}"
-    limit_e="1000" limit_l="-3.14" limit_u="3.14" limit_v="0.5" />
-  <!--LEFT_WHEEL-->
-  <m_link_mesh name="${link_02_name}"
-    origin_rpy_i="0 0 0" origin_xyz_i="0.0 0.0 0.0"
-    origin_rpy_c="0 0 0" origin_xyz_c="0 0 0"
-    origin_rpy_v = "0 0 0" origin_xyz_v ="0 0 0"
-    mass="0.02990224"
-    ixx="0.00001354" ixy="0" ixz="0"
-    iyy="0.00001354" iyz="0"
-    izz="0.00002032"
-    meshfile="package://dhex_description/meshes/wheel.dae"
-    meshscale="1 1 1" />
-  <!-- JOINT - HEX_BASE_LINK TO CASTER_WHEEL_SUPPORT -->
-  <m_joint name="${link_00_name}_TO_${link_03_name}" type="continuous"
-    axis_xyz="0 0 1"
-    origin_rpy="0 0 0" origin_xyz="-0.06827047 0.00004137 -0.03548239"
-    parent="${link_00_name}" child="${link_03_name}"
-    limit_e="1000" limit_l="-3.14" limit_u="3.14" limit_v="0.5" />
-  <!--CASTER_WHEEL_SUPPORT-->
-  <m_link_mesh name="${link_03_name}"
-    origin_rpy_i="0 0 0" origin_xyz_i="-0.00046976 -0.00666343 0.01149424"
-    origin_rpy_c="0 0 0" origin_xyz_c="0 0 0"
-    origin_rpy_v = "0 0 0" origin_xyz_v ="0 0 0"
-    mass="0.01744074 "
-    ixx="0.00000232" ixy="-7.239e-8" ixz="-9.416e-8"
-    iyy="0.00000226" iyz="-7.1e-7"
-    izz="0.0000025"
-    meshfile="package://dhex_description/meshes/caster_wheel_support.stl"
-    meshscale="1 1 1" />
-  <!-- JOINT - HEX_BASE_LINK TO CASTER_WHEEL -->
-  <m_joint name="${link_03_name}_TO_${link_04_name}" type="continuous"
-    axis_xyz="0 0 1"
-    origin_rpy="0 1.5707 0" origin_xyz="0 -0.0155 0"
-    parent="${link_03_name}" child="${link_04_name}"
-    limit_e="1000" limit_l="-3.14" limit_u="3.14" limit_v="0.5" />
-  <!--CASTER_WHEEL-->
-  <m_link_mesh name="${link_04_name}"
-    origin_rpy_i="0 0 0" origin_xyz_i="0.0 0.0 0.0"
-    origin_rpy_c="0 0 0" origin_xyz_c="0 0 0"
-    origin_rpy_v = "0 0 0" origin_xyz_v ="0 0 0"
-    mass="0.00473765"
-    ixx="2.659e-7" ixy="0" ixz="0"
-    iyy="2.659e-7" iyz="0"
-    izz="4.200e-7"
-    meshfile="package://dhex_description/meshes/caster_wheel.stl"
-    meshscale="1 1 1" />
-  <gazebo>
-		<!-- <plugin name="gazebo_ros_control" filename="libgazebo_ros_control.so">
-		</plugin> -->
-		<!-- <plugin name="gazebo_ros_control" filename="libgazebo_ros_diff_drive.so">
-			<robotNamespace>/</robotNamespace>
-			<legacyModeNS>true</legacyModeNS>
-			<alwaysOn>true</alwaysOn>
-			<legacyMode>false</legacyMode>
-			<updateRate>50</updateRate>
-			<leftJoint>${link_00_name}_TO_${link_02_name}</leftJoint>
-			<rightJoint>${link_00_name}_TO_${link_01_name}</rightJoint>
-			<wheelSeparation>0.1275</wheelSeparation>
-			<wheelDiameter>0.06599749</wheelDiameter>
-			<torque>20</torque>
-			<commandTopic>/dhex/cmd_vel</commandTopic>
-			<odometryTopic>/dhex/odom</odometryTopic>
-			<odometryFrame>odom</odometryFrame>
-			<publishWheelTF>true</publishWheelTF>
-			<publishOdomTF>true</publishOdomTF>
-			<publishWheelJointState>true</publishWheelJointState>
-			<robotBaseFrame>${base_link}</robotBaseFrame>
-		</plugin>
-    <plugin name="p3d_base_controller" filename="libgazebo_ros_p3d.so">
-      <alwaysOn>true</alwaysOn>
-      <updateRate>50.0</updateRate>
-      <bodyName>base_link</bodyName>
-      <topicName>ground_truth/state</topicName>
-      <gaussianNoise>0.01</gaussianNoise>
-      <frameName>map</frameName>
-      <xyzOffset>0 0 0</xyzOffset>
-      <rpyOffset>0 0 0</rpyOffset>
-    </plugin> -->
-	</gazebo>
+<!-- BGN - Include -->
+<xacro:include filename="$(find dhex_description)/urdf/dhex_parameters.xacro" />
+<xacro:include filename="$(find dhex_description)/urdf/links_joints.xacro" />
+<!-- END - Include -->
+<!-- BGN - Robot description -->
+<!-- BASE  -->
+<link name="${base_link}"/>
+ <!-- JOINT - BASE_LINK TO HEX_BASE_LINK -->
+<xacro:m_joint name="${base_link}_TO_${link_00_name}" type="fixed"
+  axis_xyz="0 0 1"
+  origin_rpy="0 0 0" origin_xyz="0 0 0"
+  parent="${base_link}" child="${link_00_name}"
+  limit_e="1000" limit_l="-3.14" limit_u="3.14" limit_v="0.5" />
+<!-- HEX_BASE_LINK  -->
+<xacro:m_link_mesh name="${link_00_name}"
+  origin_rpy_i="0 0 0" origin_xyz_i="0.00643363 -0.00003738 0.00608448"
+  origin_rpy_c="0 0 0" origin_xyz_c="0 0 0"
+  origin_rpy_v = "0 0 0" origin_xyz_v ="0 0 0"
+  mass="0.27625906"
+  ixx="0.0003358" ixy="2.321e-6" ixz="-3.063e-5"
+  iyy="0.00073197" iyz="0.00000108"
+  izz="0.00089429"
+  meshfile="package://dhex_description/meshes/dhex_base_link.dae"
+  meshscale="1 1 1" />
+<!-- JOINT - HEX_BASE_LINK TO RIGHT_WHEEL -->
+<xacro:m_joint name="${link_00_name}_TO_${link_01_name}" type="continuous"
+  axis_xyz="0 0 -1"
+  origin_rpy="1.5707 0 0" origin_xyz="0.04739898 -0.06196184 -0.01215966"
+  parent="${link_00_name}" child="${link_01_name}"
+  limit_e="1000" limit_l="-3.14" limit_u="3.14" limit_v="0.5" />
+<!-- RIGHT_WHEEL  -->
+<xacro:m_link_mesh name="${link_01_name}"
+  origin_rpy_i="0 0 0" origin_xyz_i="0 0 0"
+  origin_rpy_c="0 0 0" origin_xyz_c="0 0 0"
+  origin_rpy_v = "0 0 0" origin_xyz_v ="0 0 0"
+  mass="0.02990224"
+  ixx="0.00001354" ixy="0" ixz="0"
+  iyy="0.00001354" iyz="0"
+  izz="0.00002032"
+  meshfile="package://dhex_description/meshes/wheel.dae"
+  meshscale="1 1 1" />
+  <!-- origin_rpy_i="0 0 0" origin_xyz_i="0.04318327 -0.06196513 -0.0084928" -->
+<!-- JOINT - HEX_BASE_LINK TO LEFT_WHEEL -->
+<xacro:m_joint name="${link_00_name}_TO_${link_02_name}" type="continuous"
+  axis_xyz="0 0 1"
+  origin_rpy="-1.5707 0 0" origin_xyz="0.04739898 0.06196184 -0.01215966"
+  parent="${link_00_name}" child="${link_02_name}"
+  limit_e="1000" limit_l="-3.14" limit_u="3.14" limit_v="0.5" />
+<!--LEFT_WHEEL-->
+<xacro:m_link_mesh name="${link_02_name}"
+  origin_rpy_i="0 0 0" origin_xyz_i="0.0 0.0 0.0"
+  origin_rpy_c="0 0 0" origin_xyz_c="0 0 0"
+  origin_rpy_v = "0 0 0" origin_xyz_v ="0 0 0"
+  mass="0.02990224"
+  ixx="0.00001354" ixy="0" ixz="0"
+  iyy="0.00001354" iyz="0"
+  izz="0.00002032"
+  meshfile="package://dhex_description/meshes/wheel.dae"
+  meshscale="1 1 1" />
+<!-- JOINT - HEX_BASE_LINK TO CASTER_WHEEL_SUPPORT -->
+<xacro:m_joint name="${link_00_name}_TO_${link_03_name}" type="continuous"
+  axis_xyz="0 0 1"
+  origin_rpy="0 0 0" origin_xyz="-0.06827047 0.00004137 -0.03548239"
+  parent="${link_00_name}" child="${link_03_name}"
+  limit_e="1000" limit_l="-3.14" limit_u="3.14" limit_v="0.5" />
+<!--CASTER_WHEEL_SUPPORT-->
+<xacro:m_link_mesh name="${link_03_name}"
+  origin_rpy_i="0 0 0" origin_xyz_i="-0.00046976 -0.00666343 0.01149424"
+  origin_rpy_c="0 0 0" origin_xyz_c="0 0 0"
+  origin_rpy_v = "0 0 0" origin_xyz_v ="0 0 0"
+  mass="0.01744074 "
+  ixx="0.00000232" ixy="-7.239e-8" ixz="-9.416e-8"
+  iyy="0.00000226" iyz="-7.1e-7"
+  izz="0.0000025"
+  meshfile="package://dhex_description/meshes/caster_wheel_support.stl"
+  meshscale="1 1 1" />
+<!-- JOINT - HEX_BASE_LINK TO CASTER_WHEEL -->
+<xacro:m_joint name="${link_03_name}_TO_${link_04_name}" type="continuous"
+  axis_xyz="0 0 1"
+  origin_rpy="0 1.5707 0" origin_xyz="0 -0.0155 0"
+  parent="${link_03_name}" child="${link_04_name}"
+  limit_e="1000" limit_l="-3.14" limit_u="3.14" limit_v="0.5" />
+<!--CASTER_WHEEL-->
+<xacro:m_link_mesh name="${link_04_name}"
+  origin_rpy_i="0 0 0" origin_xyz_i="0.0 0.0 0.0"
+  origin_rpy_c="0 0 0" origin_xyz_c="0 0 0"
+  origin_rpy_v = "0 0 0" origin_xyz_v ="0 0 0"
+  mass="0.00473765"
+  ixx="2.659e-7" ixy="0" ixz="0"
+  iyy="2.659e-7" iyz="0"
+  izz="4.200e-7"
+  meshfile="package://dhex_description/meshes/caster_wheel.stl"
+  meshscale="1 1 1" />
 </robot>

File: dhex_description/urdf/links_joints.xacro (robot description, xacro)
@@ -54,5 +54,4 @@
           <mesh filename="${meshfile}" scale="${meshscale}"/>
         </geometry>
-        <material name="light_black"/>
       </visual>
     </link>
