Commit message: Add ros_control to controle wheel velocities

File: dhex_description/urdf/dhex.urdf.xacro (robot description, xacro)
@@ -10,8 +10,9 @@
  <!-- JOINT - BASE_LINK TO HEX_BASE_LINK -->
 <xacro:m_joint name="${base_link}_TO_${link_00_name}" type="fixed"
+  motor_flag = "false"
   axis_xyz="0 0 1"
   origin_rpy="0 0 0" origin_xyz="0 0 0"
   parent="${base_link}" child="${link_00_name}"
-  limit_e="1000" limit_l="-3.14" limit_u="3.14" limit_v="0.5" />
+  limit_e="100000" limit_l="-100000" limit_u="1000000" limit_v="10"/>
 <!-- HEX_BASE_LINK  -->
 <xacro:m_link_mesh name="${link_00_name}"
@@ -27,8 +28,20 @@
 <!-- JOINT - HEX_BASE_LINK TO RIGHT_WHEEL -->
 <xacro:m_joint name="${link_00_name}_TO_${link_01_name}" type="continuous"
+  motor_flag = "true"
   axis_xyz="0 0 -1"
   origin_rpy="1.5707 0 0" origin_xyz="0.04739898 -0.06196184 -0.01215966"
   parent="${link_00_name}" child="${link_01_name}"
-  limit_e="1000" limit_l="-3.14" limit_u="3.14" limit_v="0.5" />
+  limit_e="100000" limit_l="-100000" limit_u="1000000" limit_v="10"/>
+<!--TODO: Understand why the macro is not working-->
+<transmission name="trans_${link_00_name}_TO_${link_01_name}">
+  <type>transmission_interface/SimpleTransmission</type>
+  <joint name="${link_00_name}_TO_${link_01_name}">
+    <hardwareInterface>hardware_interface/EffortJointInterface</hardwareInterface>
+  </joint>
+  <actuator name="motor_${link_00_name}_TO_${link_01_name}">
+    <hardwareInterface>hardware_interface/EffortJointInterface</hardwareInterface>
+    <mechanicalReduction>1</mechanicalReduction>
+  </actuator>
+</transmission>
 <!-- RIGHT_WHEEL  -->
 <xacro:m_link_mesh name="${link_01_name}"
@@ -45,8 +58,20 @@
 <!-- JOINT - HEX_BASE_LINK TO LEFT_WHEEL -->
 <xacro:m_joint name="${link_00_name}_TO_${link_02_name}" type="continuous"
+  motor_flag = "true"
   axis_xyz="0 0 1"
   origin_rpy="-1.5707 0 0" origin_xyz="0.04739898 0.06196184 -0.01215966"
   parent="${link_00_name}" child="${link_02_name}"
-  limit_e="1000" limit_l="-3.14" limit_u="3.14" limit_v="0.5" />
+  limit_e="100000" limit_l="-100000" limit_u="1000000" limit_v="10"/>
+<!--TODO: Understand why the macro is not working-->
+<transmission name="trans_${link_00_name}_TO_${link_02_name}">
+  <type>transmission_interface/SimpleTransmission</type>
+  <joint name="${link_00_name}_TO_${link_02_name}">
+    <hardwareInterface>hardware_interface/EffortJointInterface</hardwareInterface>
+  </joint>
+  <actuator name="motor_${link_00_name}_TO_${link_02_name}">
+    <hardwareInterface>hardware_interface/EffortJointInterface</hardwareInterface>
+    <mechanicalReduction>1</mechanicalReduction>
+  </actuator>
+</transmission>
 <!--LEFT_WHEEL-->
 <xacro:m_link_mesh name="${link_02_name}"
@@ -62,8 +87,9 @@
 <!-- JOINT - HEX_BASE_LINK TO CASTER_WHEEL_SUPPORT -->
 <xacro:m_joint name="${link_00_name}_TO_${link_03_name}" type="continuous"
+  motor_flag = "false"
   axis_xyz="0 0 1"
   origin_rpy="0 0 0" origin_xyz="-0.06827047 0.00004137 -0.03548239"
   parent="${link_00_name}" child="${link_03_name}"
-  limit_e="1000" limit_l="-3.14" limit_u="3.14" limit_v="0.5" />
+  limit_e="100000" limit_l="-100000" limit_u="1000000" limit_v="10"/>
 <!--CASTER_WHEEL_SUPPORT-->
 <xacro:m_link_mesh name="${link_03_name}"
@@ -79,4 +105,5 @@
 <!-- JOINT - HEX_BASE_LINK TO CASTER_WHEEL -->
 <xacro:m_joint name="${link_03_name}_TO_${link_04_name}" type="continuous"
+  motor_flag = "false"
   axis_xyz="0 0 1"
   origin_rpy="0 1.5707 0" origin_xyz="0 -0.0155 0"
@@ -94,3 +121,9 @@
   meshfile="package://dhex_description/meshes/caster_wheel.stl"
   meshscale="1 1 1" />
+  <gazebo>
+    <plugin name="gazebo_ros_control" filename="libgazebo_ros_control.so">
+      <robotNamespace>/dhex</robotNamespace>
+      <!-- <robotSimType>gazebo_ros_control/DefaultRobotHWSim</robotSimType> -->
+    </plugin>
+  </gazebo>
 </robot>

File: dhex_description/urdf/links_joints.xacro (robot description, xacro)
@@ -1,5 +1,8 @@
 <?xml version="1.0" ?>
 <robot xmlns:xacro="http://www.ros.org/wiki/xacro">
-  <xacro:macro name="m_joint" params="name type motor_flag:=false axis_xyz origin_rpy origin_xyz parent child limit_e limit_l limit_u limit_v">
+  <xacro:macro name="m_joint" params="name type motor_flag axis_xyz origin_rpy origin_xyz parent child limit_e limit_l limit_u limit_v">
+  <xacro:property name="revolute_type" value="revolute"/>
+  <xacro:property name="continuos_type" value="continuos"/>
+  <xacro:property name="true_bool" value="true"/>
     <joint name="${name}" type="${type}">
       <axis xyz="${axis_xyz}" />
@@ -9,6 +12,6 @@
       <child link="${child}" />
     </joint>
-  <xacro:if value="${motor_flag == 'true'}">
-    <xacro:if value="${joint_type == 'revolute'}">
+  <xacro:if value="${motor_flag == true_bool}">
+    <xacro:if value="${type == revolute_type}">
       <transmission name="trans_${name}">
         <type>transmission_interface/SimpleTransmission</type>
@@ -22,12 +25,12 @@
       </transmission>
     </xacro:if>
-    <xacro:if value="${joint_type == 'continuous'}">
+    <xacro:if value="${type == continuos_type}">
       <transmission name="trans_${name}">
         <type>transmission_interface/SimpleTransmission</type>
         <joint name="${name}">
-          <hardwareInterface>hardware_interface/VelocityJointInterface</hardwareInterface>
+          <hardwareInterface>hardware_interface/EffortJointInterface</hardwareInterface>
         </joint>
         <actuator name="motor_${name}">
-          <hardwareInterface>hardware_interface/VelocityJointInterface</hardwareInterface>
+          <hardwareInterface>hardware_interface/EffortJointInterface</hardwareInterface>
           <mechanicalReduction>1</mechanicalReduction>
         </actuator>
